File: Mini_VME_Backplane/Mini_VME_Backplane/sockets1.kicad_sch (KiCad schematic)
At the start: 13 parts, among them U1 74HCT1G32, U2 74HCT1G32, U3 74HCT1G32, U4 74HCT1G32, U5 74HCT1G32, X1 DIN41612_03x32_ABC_VMEbus, X2 DIN41612_03x32_ABC_VMEbus, X3 DIN41612_03x32_ABC_VMEbus

Commit message: As ordered Apr 27
Parts:
- removed R1, R2, R3, R4, R5: 10K, COMET_footprints:R_SMD0805, symbol COMET Symbols:R
- removed U1, U2, U3, U4, U5: 74HCT1G32, COMET_footprints:Package_SOT23-5, symbol COMET Symbols:74x1G32
- removed X3: DIN41612_03x32_ABC_VMEbus, Connector_DIN:DIN41612_C_3x32_Male_Horizontal_THT, symbol COMET Symbols:DIN41612_03x32_ABC_VMEbus
- added J1: Screw_Terminal_01x05, TerminalBlock_Phoenix:TerminalBlock_Phoenix_MKDS-1,5-5-5.08_1x05_P5.08mm_Horizontal, symbol Connector:Screw_Terminal_01x05
- X1, X2: footprint Connector_DIN:DIN41612_C_3x32_Male_Horizontal_THT -> Connector_DIN:DIN41612_C_3x32_Female_Vertical_THT
Connections:
- net +12V: now also J1.4 (Pin_4)
- net +5V: now also J1.1 (Pin_1)
- net -12V: now also J1.5 (Pin_5)
- net D8: no longer X1.a9 (GND), X2.a9 (GND)
- net GND: now also X1.a9 (GND), X2.a9 (GND), J1.3 (Pin_3)
- net +5VSTDBY renamed +5VA
- net +5VA: now also J1.2 (Pin_2)
- net ~{BG0OUT_2}: no longer names the net of X2.b5 (~{BG0OUT})
- net ~{BG1OUT_2}: no longer names the net of X2.b7 (~{BG1OUT})
- net ~{BG2OUT_2}: no longer names the net of X2.b9 (~{BG2OUT})
- net ~{BG3OUT_2}: no longer names the net of X2.b11 (~{BG3OUT})
- net ~{IACKOUT_2}: no longer names the net of X2.a22 (~{IACKOUT})
Other:
- note added: "SLOT 1"
- note added: "SLOT 2"
- moved on the sheet: X1A, X1B, X1C, X2A, X2B, X2C
