File: VME_Protoboard_160/VME_Protoboard_160/VME_Protoboard_160.kicad_sch (KiCad schematic)
At the start: 95 parts, among them J1 Conn_02x04_Odd_Even, J2 Conn_02x04_Odd_Even, J3 Conn_02x07_Odd_Even, U1 74x16245, U2 74x16245, U3 74x16245, U4 74x1G19, U5 74x1G07, U6 74x1G07, U7 74x1G125, U8 74x1G125, U9 74x1G125, X1 DIN41612_03x32_ABC_VMEbus

Commit message: Very nearly complete, just need to organise component labels etc
Parts:
- removed J1, J2: Conn_02x04_Odd_Even, Connector_PinHeader_2.54mm:PinHeader_2x04_P2.54mm_Vertical, symbol Connector_Generic:Conn_02x04_Odd_Even
- removed TP1, TP10, TP11, TP12, TP14, TP15, TP16, TP2, TP20, TP21, TP22, TP23, TP24, TP25, TP26, TP27, TP28, TP29, TP3, TP30, TP31, TP32, TP33, TP34, TP35, TP36, TP37, TP38, TP39, TP4, TP40, TP41, TP42, TP43, TP44, TP45, TP46, TP47, TP48, TP49, TP5, TP8, TP9: TestPoint, TestPoint:TestPoint_Loop_D1.80mm_Drill1.0mm_Beaded, symbol Connector:TestPoint
- added C12: 100uF, COMET_footprints:C_SMD_4.3MMx7.3MM, symbol Device:C_Polarized
- added J1: Conn_02x08_Odd_Even, Connector_PinHeader_2.54mm:PinHeader_2x08_P2.54mm_Vertical, symbol Connector_Generic:Conn_02x08_Odd_Even
- added J2: Conn_02x08_Odd_Even, Connector_PinHeader_2.54mm:PinHeader_2x07_P2.54mm_Vertical, symbol Connector_Generic:Conn_02x07_Odd_Even
- added J3: Conn_02x12_Odd_Even, Connector_PinHeader_2.54mm:PinHeader_2x12_P2.54mm_Vertical, symbol Connector_Generic:Conn_02x12_Odd_Even
- added R7: 10K, COMET_footprints:R_SMD0805, symbol COMET_symbols:R
- renumbered C12 to C13, C13 to C14, C14 to C15, C15 to C16, J3 to J4, TP17 to TP1, TP54 to TP10, TP55 to TP11, TP56 to TP12, TP18 to TP2, TP19 to TP3, TP50 to TP4, TP51 to TP5, TP52 to TP8, TP53 to TP9
Connections:
- net +5V: now also C12.1, R7.2
- net D0: now also J1.1 (Pin_1)
- net D1: now also J1.3 (Pin_3); no longer TP13.1
- net D10: now also J1.6 (Pin_6)
- net D11: now also J1.8 (Pin_8)
- net D12: now also J1.10 (Pin_10)
- net D13: now also J1.12 (Pin_12); no longer TP6.1
- net D14: now also J1.14 (Pin_14)
- net D15: now also J1.16 (Pin_16)
- net D2: now also J1.5 (Pin_5)
- net D3: now also J1.7 (Pin_7)
- net D4: now also J1.9 (Pin_9); no longer TP7.1
- net D5: now also J1.11 (Pin_11)
- net D6: now also J1.13 (Pin_13)
- net D7: now also J1.15 (Pin_15)
- net D8: now also J1.2 (Pin_2)
- net D9: now also J1.4 (Pin_4)
- net GND: now also C12.2, J2.1 (Pin_1), J2.11 (Pin_11), J2.13 (Pin_13), J2.3 (Pin_3), J2.5 (Pin_5), J2.7 (Pin_7), J2.9 (Pin_9), J3.15 (Pin_15)
- net ~{BERR`}: now also TP7.1
- net ~{DTACK`}: now also TP6.1
- net ~{IRQ1`}: now also J4.1 (Pin_1); no longer J4.14 (Pin_14)
- net ~{IRQ2`}: now also J4.3 (Pin_3); no longer J4.12 (Pin_12)
- net ~{IRQ3`}: now also J4.5 (Pin_5); no longer J4.10 (Pin_10)
- net ~{IRQ4`}: now also J4.7 (Pin_7); no longer J4.8 (Pin_8)
- net ~{IRQ5`}: now also J4.9 (Pin_9); no longer J4.6 (Pin_6)
- net ~{IRQ6`}: now also J4.11 (Pin_11); no longer J4.4 (Pin_4)
- net ~{IRQ7`}: now also J4.13 (Pin_13); no longer J4.2 (Pin_2)
- net ~{IRQ}: now also R7.1
- net A12: now reaches U2.35 (2A2)
- net A12: now also J3.10 (Pin_10)
- net ~{UDS}: now reaches U3.27 (2A7)
- net ~{UDS}: now also J2.14 (Pin_14)
- net ~{LDS}: now reaches U3.29 (2A6)
- net ~{LDS}: now also J2.12 (Pin_12)
- net ~{WRITE}: now reaches U3.30 (2A5)
- net ~{WRITE}: now also J2.10 (Pin_10)
- net A23: now reaches U3.32 (2A4)
- net A23: now also J3.24 (Pin_24)
- net FC0: now reaches U3.33 (2A3)
- net FC0: now also J2.8 (Pin_8)
- net A22: now reaches U3.35 (2A2)
- net A22: now also J3.23 (Pin_23)
- net FC1: now reaches U3.36 (2A1)
- net FC1: now also J2.6 (Pin_6)
- net ~{AS}: now reaches U3.41 (1A5)
- net ~{AS}: now also J2.2 (Pin_2)
- net A16: now reaches U3.47 (1A1)
- net A16: now also J3.17 (Pin_17)
- net at U8.4: now also TP13.1
- net A15: now reaches U2.27 (2A7)
- net A15: now also J3.16 (Pin_16)
- net A14: now reaches U2.29 (2A6)
- net A14: now also J3.14 (Pin_14)
- net A7: now reaches U2.30 (2A5)
- net A7: now also J3.13 (Pin_13)
- net A13: now reaches U2.32 (2A4)
- net A13: now also J3.12 (Pin_12)
- net A6: now reaches U2.33 (2A3)
- net A6: now also J3.11 (Pin_11)
- net A5: now reaches U2.36 (2A1)
- net A5: now also J3.9 (Pin_9)
- net A2: now reaches U2.44 (1A3)
- net A2: now also J3.3 (Pin_3)
- net A20: now reaches U3.40 (1A6)
- net A20: now also J3.21 (Pin_21)
- net A10: now reaches U2.40 (1A6)
- net A10: now also J3.6 (Pin_6)
- net A1: now reaches U2.47 (1A1)
- net A1: now also J3.1 (Pin_1)
- net A4: now reaches U2.38 (1A7)
- net A4: now also J3.7 (Pin_7)
- net A8: now reaches U2.46 (1A2)
- net A8: now also J3.2 (Pin_2)
- net A18: now reaches U3.44 (1A3)
- net A18: now also J3.19 (Pin_19)
- net FC2: now reaches U3.38 (1A7)
- net FC2: now also J2.4 (Pin_4)
- net A11: now reaches U2.37 (1A8)
- net A11: now also J3.8 (Pin_8)
- net A9: now reaches U2.43 (1A4)
- net A9: now also J3.4 (Pin_4)
- net A17: now reaches U3.46 (1A2)
- net A17: now also J3.18 (Pin_18)
- net A3: now reaches U2.41 (1A5)
- net A3: now also J3.5 (Pin_5)
- net A19: now reaches U3.43 (1A4)
- net A19: now also J3.20 (Pin_20)
- net A21: now reaches U3.37 (1A8)
- net A21: now also J3.22 (Pin_22)
- net ~{BERR} renamed ~{BERR_DRV}
- net ~{DTACK} renamed ~{DTACK_DRV}
- new net: J4.10 (Pin_10), J4.12 (Pin_12), J4.14 (Pin_14), J4.2 (Pin_2), J4.4 (Pin_4), J4.6 (Pin_6), J4.8 (Pin_8), U9.4
Other:
- moved on the sheet: J4, U9A
