File: VME_Backplane_8ActPas/slot3.kicad_sch (KiCad schematic)
At the start: 7 parts, among them X103 DIN41612_03x32_ABC_VMEbus, X403A1 Jumper_2_Open, X403B1 Jumper_2_Open, X403C1 Jumper_2_Open, X403D1 Jumper_2_Open, X503 Jumper_2_Open

Commit message: Fix page names
Other:
- title: SLOT 2 -> SLOT 3
Changed lines of the file:
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@@
   (paper "A4")
   (title_block
-    (title "SLOT 2")
+    (title "SLOT 3")
     (date "2024-01-04")
     (rev "1")
