File: VME_Backplane_8ActPas/slot6.kicad_sch (KiCad schematic)
At the start: 7 parts, among them X106 DIN41612_03x32_ABC_VMEbus, X406A1 Jumper_2_Open, X406B1 Jumper_2_Open, X406C1 Jumper_2_Open, X406D1 Jumper_2_Open, X506 Jumper_2_Open

Commit message: Fix page names
Other:
- title: SLOT 2 -> SLOT 6
Changed lines of the file:
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@@
   (paper "A4")
   (title_block
-    (title "SLOT 2")
+    (title "SLOT 6")
     (date "2024-01-04")
     (rev "1")
