File: VME_Backplane_8ActPas/slot8.kicad_sch (KiCad schematic)
At the start: 2 parts, among them X108 DIN41612_03x32_ABC_VMEbus

Commit message: Fix page names
Other:
- title: SLOT 3 -> SLOT 8
Changed lines of the file:
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@@
   (paper "A4")
   (title_block
-    (title "SLOT 3")
+    (title "SLOT 8")
     (date "2024-01-04")
     (rev "1")
