File: Video_Card/fpga_regen.kicad_sch (KiCad schematic)
At the start: 4 parts, among them U7 EPF81188AQC208-3

Commit message: Final work for rev 1
Parts:
- removed U7: EPF81188AQC208-3, COMET_footprints:Package_PQFP-208_28x28mm_P0.5mm, symbol Video_Card:FPGA_dev
- added R23: 10K, COMET_footprints:R_SMD0805, symbol COMET_symbols:R
- added RN10, RN11, RN12, RN13: 10K, COMET_footprints:R_Cat16-4, symbol Device:R_Pack04
- added U5: EPF81188AQC208-3, COMET_footprints:Package_PQFP-208_28x28mm_P0.5mm, symbol Video_Card:EPF81188AQC208-3
- RN4: renamed from RN6; footprint Resistor_SMD:R_Cat16-4 -> COMET_footprints:R_Cat16-4
- renumbered R27 to R22, R28 to R24
Connections:
- net +5V: now also R23.1, RN10.5 (R4.2), RN10.6 (R3.2), RN10.7 (R2.2), RN10.8 (R1.2), RN11.5 (R4.2), RN11.6 (R3.2), RN11.7 (R2.2), RN11.8 (R1.2), RN12.5 (R4.2), RN12.6 (R3.2), RN12.7 (R2.2), RN12.8 (R1.2), RN13.5 (R4.2), RN13.6 (R3.2), RN13.7 (R2.2), RN13.8 (R1.2)
- net BMUX_S0: now also U5.56 (BMUX_S0)
- net BMUX_S1: now also U5.194 (BMUX_S1)
- net BMUX_S2: now also U5.206 (BMUX_S2)
- net FONTSEL: now also U5.26 (FONTSEL)
- net MA1: now also U5.10 (MA0)
- net MA10: now also U5.30 (MA9)
- net MA11: now also U5.205 (MA10)
- net MA12: now also U5.61 (MA11)
- net MA13: now also U5.125 (MA12)
- net MA14: now also U5.135 (MA13)
- net MA15: now also U5.92 (MA14)
- net MA16: now also U5.141 (MA15)
- net MA2: now also U5.127 (MA1)
- net MA3: now also U5.128 (MA2)
- net MA4: now also U5.64 (MA3)
- net MA5: now also U5.196 (MA4)
- net MA6: now also U5.130 (MA5)
- net MA7: now also U5.137 (MA6)
- net MA8: now also U5.24 (MA7)
- net MA9: now also U5.134 (MA8)
- net MD0: now also RN10.4 (R4.1), U5.108 (MD0)
- net MD1: now also RN10.3 (R3.1), U5.113 (MD1)
- net MD10: now also RN12.3 (R3.1), U5.97 (MD10)
- net MD11: now also RN12.4 (R4.1), U5.175 (MD11)
- net MD12: now also RN13.1 (R1.1), U5.59 (MD12)
- net MD13: now also RN13.2 (R2.1), U5.109 (MD13)
- net MD14: now also RN13.3 (R3.1), U5.73 (MD14)
- net MD15: now also RN13.4 (R4.1), U5.74 (MD15)
- net MD2: now also RN10.2 (R2.1), U5.190 (MD2)
- net MD3: now also RN10.1 (R1.1), U5.112 (MD3)
- net MD4: now also RN11.4 (R4.1), U5.71 (MD4)
- net MD5: now also RN11.3 (R3.1), U5.110 (MD5)
- net MD6: now also RN11.2 (R2.1), U5.47 (MD6)
- net MD7: now also RN11.1 (R1.1), U5.46 (MD7)
- net MD8: now also RN12.1 (R1.1), U5.70 (MD8)
- net MD9: now also RN12.2 (R2.1), U5.89 (MD9)
- net RA0: now also U5.79 (RA0)
- net RA1: now also U5.184 (RA1)
- net RA2: now also U5.136 (RA2)
- net RA3: now also U5.25 (RA3)
- net ~{REGEN_CS}: now also U5.68 (~{REGEN_CS})
- net B0SEL: no longer names the net of RN4.5 (R4.2)
- new net FD0: U5.83 (FD0)
- new net FD1: U5.171 (FD1)
- new net FD2: U5.173 (FD2)
- new net FD3: U5.180 (FD3)
- new net FD4: U5.150 (FD4)
- new net FD5: U5.9 (FD5)
- new net FD6: U5.67 (FD6)
- new net FD7: U5.200 (FD7)
- new net ~{BANK_CS}: R23.2, U5.169 (~{BANK_CS})
- no-connect marks 0 -> 2
Other:
- moved on the sheet: R22, R24, RN4
