File: Video_Card/i2c.kicad_sch (KiCad schematic)
At the start: 10 parts, among them U24 PCF8584T, U7 EPF81188AQC208-3

Commit message: Final work for rev 1
Parts:
- removed C6: 100nF, COMET_footprints:C_SMD0805, symbol COMET_symbols:C
- removed unit 2 of U24
- removed U7: EPF81188AQC208-3, COMET_footprints:Package_PQFP-208_28x28mm_P0.5mm, symbol Video_Card:FPGA_dev
- added U5: EPF81188AQC208-3, COMET_footprints:Package_PQFP-208_28x28mm_P0.5mm, symbol Video_Card:EPF81188AQC208-3
- renumbered R35 to R49, R33 to R50, R34 to R51, R30 to R52, R31 to R53, R32 to R54, R29 to R55, U24 to U21
Connections:
- net at R52.1, U21.17 (~{CS}): now also U5.143 (~{CS})
- net at R49.1, U21.19 (~{RESET}): now also U5.172 (~{RESET})
- net at U21.1 (CLK): now also U5.8 (CLK)
- net at R53.1, U21.16 (~{DTACK}): now also U5.166 (~{DTACK})
- net at R54.1, U21.5 (~{INT}): now also U5.93 (~{INT})
- net XA0 renamed A1
- net XD0 renamed D8
- net XD1 renamed D9
- net XD2 renamed D10
- net XD3 renamed D11
- net XD4 renamed D12
- net XD5 renamed D13
- net XD6 renamed D14
- net XD7 renamed D15
