File: Video_Card/regen_bus_mux_1.kicad_sch (KiCad schematic)
At the start: 1 part, among them U16 SN74CBT16212CDLR

Commit message: Final work for rev 1
Parts:
- removed unit 2 of U16
- renumbered U16 to U11
Connections:
- net B0D0 is gone; now on net B0D4: U11.54 (1B1)
- net B0D1 is gone; now on net B0D5: U11.52 (2B1)
- net B0D2 is gone; now on net B0D6: U11.50 (3B1)
- net B0D3 is gone; now on net B0D7: U11.47 (4B1)
- net B1D0 is gone; now on net B1D4: U11.53 (1B2)
- net B1D1 is gone; now on net B1D5: U11.51 (2B2)
- net B1D2 is gone; now on net B1D6: U11.48 (3B2)
- net B2D3 is gone; now on net B1D7: U11.46 (4B2)
- net D0 is gone; now on net D4: U11.2 (1A1)
- net D1 is gone; now on net D5: U11.4 (2A1)
- net D2 is gone; now on net D6: U11.6 (3A1)
- net D3 is gone; now on net D7: U11.9 (4A1)
- net MD0 is gone; now on net MD4: U11.3 (1A2)
- net MD1 is gone; now on net MD5: U11.5 (2A2)
- net MD2 is gone; now on net MD6: U11.7 (3A2)
- net MD3 is gone; now on net MD7: U11.10 (4A2)
- net B0D10: now also U11.34 (10B1); no longer U11.32 (11B1)
- net B0D11: now also U11.36 (9B1); no longer U11.30 (12B1)
- net B0D4: no longer U11.45 (5B1)
- net B0D5: no longer U11.43 (6B1)
- net B0D6: no longer U11.41 (7B1)
- net B0D7: no longer U11.39 (8B1)
- net B0D8: now also U11.30 (12B1); no longer U11.36 (9B1)
- net B0D9: now also U11.32 (11B1); no longer U11.34 (10B1)
- net B1D10: now also U11.33 (10B2); no longer U11.31 (11B2)
- net B1D11: now also U11.35 (9B2); no longer U11.29 (12B2)
- net B1D4: no longer U11.44 (5B2)
- net B1D5: no longer U11.42 (6B2)
- net B1D6: no longer U11.40 (7B2)
- net B1D7: no longer U11.37 (8B2)
- net B1D8: now also U11.29 (12B2); no longer U11.35 (9B2)
- net B1D9: now also U11.31 (11B2); no longer U11.33 (10B2)
- net D10: now also U11.23 (10A1); no longer U11.25 (11A1)
- net D11: now also U11.21 (9A1); no longer U11.27 (12A1)
- net D4: no longer U11.11 (5A1)
- net D5: no longer U11.13 (6A1)
- net D6: no longer U11.15 (7A1)
- net D7: no longer U11.18 (8A1)
- net D8: now also U11.27 (12A1); no longer U11.21 (9A1)
- net D9: now also U11.25 (11A1); no longer U11.23 (10A1)
- net MD10: now also U11.24 (10A2); no longer U11.26 (11A2)
- net MD11: now also U11.22 (9A2); no longer U11.28 (12A2)
- net MD4: no longer U11.12 (5A2)
- net MD5: no longer U11.14 (6A2)
- net MD6: no longer U11.16 (7A2)
- net MD7: no longer U11.20 (8A2)
- net MD8: now also U11.28 (12A2); no longer U11.22 (9A2)
- net MD9: now also U11.26 (11A2); no longer U11.24 (10A2)
- new net B0D12: U11.39 (8B1)
- new net B0D13: U11.41 (7B1)
- new net B0D14: U11.43 (6B1)
- new net B0D15: U11.45 (5B1)
- new net B1D12: U11.37 (8B2)
- new net B1D13: U11.40 (7B2)
- new net B1D14: U11.42 (6B2)
- new net B1D15: U11.44 (5B2)
- new net D12: U11.18 (8A1)
- new net D13: U11.15 (7A1)
- new net D14: U11.13 (6A1)
- new net D15: U11.11 (5A1)
- new net MD12: U11.20 (8A2)
- new net MD13: U11.16 (7A2)
- new net MD14: U11.14 (6A2)
- new net MD15: U11.12 (5A2)
