File: Video_Card/regen_bus_mux_2.kicad_sch (KiCad schematic)
At the start: 1 part, among them U17 SN74CBT16212CDLR

Commit message: Final work for rev 1
Parts:
- removed unit 2 of U17
- added RN5, RN6: 10K, COMET_footprints:R_Cat16-4, symbol Device:R_Pack04
- renumbered U17 to U12
Connections:
- net B0D15 is gone; now on net B0A8: U12.47 (4B1)
- net B1D12 is gone; now on net B1A4: U12.53 (1B2)
- net B1D13 is gone; now on net B1A5: U12.51 (2B2)
- net B1D14 is gone; now on net B1A6: U12.48 (3B2)
- net B1D15 is gone; now on net B1A7: U12.46 (4B2)
- net D12 is gone; now on net A4: U12.2 (1A1)
- net D13 is gone; now on net A3: U12.4 (2A1)
- net D14 is gone; now on net A2: U12.6 (3A1)
- net D15 is gone; now on net A1: U12.9 (4A1)
- net MD12 is gone; now on net MA4: U12.3 (1A2)
- net MD13 is gone; now on net MA3: U12.5 (2A2)
- net MD14 is gone; now on net MA2: U12.7 (3A2)
- net MD15 is gone; now on net MA1: U12.10 (4A2)
- net A1: no longer U12.11 (5A1)
- net A2: no longer U12.13 (6A1)
- net A3: no longer U12.15 (7A1)
- net A4: no longer U12.18 (8A1)
- net B0A8: no longer U12.30 (12B1)
- net B1A4: no longer U12.37 (8B2)
- net B1A5: no longer U12.35 (9B2)
- net B1A6: no longer U12.33 (10B2)
- net B1A7: no longer U12.31 (11B2)
- net MA1: no longer U12.12 (5A2)
- net MA2: no longer U12.14 (6A2)
- net MA3: no longer U12.16 (7A2)
- net MA4: no longer U12.20 (8A2)
- net A5 renamed D0
- net A6 renamed D1
- net A7 renamed D2
- net A8 renamed D3
- net B0A1 renamed ~{B0UDS}
- net ~{B0UDS}: now also RN5.1 (R1.1)
- net B0A2 renamed ~{B0LDS}
- net ~{B0LDS}: now also RN5.2 (R2.1)
- net B0A3 renamed ~{B0WRITE}
- net ~{B0WRITE}: now also RN5.3 (R3.1)
- net B0A4 renamed ~{B0CS}
- net ~{B0CS}: now also RN5.4 (R4.1)
- net B0A5 renamed B0D0
- net B0A6 renamed B0D1
- net B0A7 renamed B0D2
- net B0D12 renamed B0A9
- net B0D13 renamed B0A10
- net B0D14 renamed B0A11
- net B1A1 renamed ~{B1UDS}
- net ~{B1UDS}: now also RN6.1 (R1.1)
- net B1A2 renamed ~{B1LDS}
- net ~{B1LDS}: now also RN6.2 (R2.1)
- net B1A3 renamed ~{B1WRITE}
- net ~{B1WRITE}: now also RN6.3 (R3.1)
- net B1A8 renamed B1D3
- net MA5 renamed MD0
- net MA6 renamed MD1
- net MA7 renamed MD2
- net MA8 renamed MD3
- new net +5V: RN5.5 (R4.2), RN5.6 (R3.2), RN5.7 (R2.2), RN5.8 (R1.2), RN6.5 (R4.2), RN6.6 (R3.2), RN6.7 (R2.2), RN6.8 (R1.2), U12.16 (7A2)
- new net B0D3: U12.30 (12B1)
- new net B1D0: U12.35 (9B2)
- new net B1D1: U12.33 (10B2)
- new net B1D2: U12.31 (11B2)
- new net GND: U12.12 (5A2), U12.14 (6A2)
- new net ~{B1CS}: RN6.4 (R4.1), U12.37 (8B2)
- new net ~{BANK_CS}: U12.20 (8A2)
- new net ~{LDS}: U12.13 (6A1)
- new net ~{REGEN_CS}: U12.18 (8A1)
- new net ~{UDS}: U12.11 (5A1)
- new net ~{WRITE}: U12.15 (7A1)
Other:
- note added: "REGEN MEMORY CONTROL SIGNALS CRTC AND FORMATTER: ~{WRITE} IS DRIVEN HIGH BECAUSE THE CRTC ONLY EVER READS FROM REGEN MEMORY ~{xDS} ARE DRIVEN LOW TO FORCE WORD READS FROM REGEN MEMORY CPU: SIGNALS ARE DRIVEN ACCORDING TO THE BUS CYCLE BEING EXECUTED"
