File: Video_Card/regen_mem.kicad_sch (KiCad schematic)
At the start: 5 parts, among them U19 IS61C6416AL-12TLI, U20 IS61C6416AL-12TLI, U21 SN74LVC1G19DBV, U22 IS61C6416AL-12TLI

Commit message: Work to date
So much to list ....

* Changed expansion ROM to 16 bit wide to remove some components
* Tried moving peripherals over to an 8 bit dedicated bus, but will have to revert this to reduce component count
* Fleshed out keyboard and I2C controller circuits
* Tried to fit in a font RAM, but I am 50/50 whether this will stick

And a lot more I am sure.
Parts:
- added U23: SST39SF010A-70-4C-NHE, COMET_footprints:Package_PLCC-32_SMD_socket, symbol COMET_symbols:39SF040
Connections:
- net +5V: now also U23.31 (~{WE}), U23.32 (VCC)
- net B0D10: now also U23.6 (A6)
- net B0D11: now also U23.5 (A7)
- net B0D12: now also U23.27 (A8)
- net B0D13: now also U23.26 (A9)
- net B0D14: now also U23.23 (A10)
- net B0D15: now also U23.25 (A11)
- net B0D8: now also U23.8 (A4)
- net B0D9: now also U23.7 (A5)
- net GND: now also U23.1 (A18), U23.16 (GND), U23.2 (A16), U23.22 (~{CE}), U23.24 (~{OE}), U23.28 (A13), U23.29 (A14), U23.3 (A15), U23.30 (A17)
- net at U20.6 (~{CE}), U21.4 (~{Y1}): no longer R26.2
- net at U19.6 (~{CE}), U21.6 (~{Y0}): now also R26.2
- new net FONTSEL: U23.4 (A12)
- new net PD0: U23.13 (D0)
- new net PD1: U23.14 (D1)
- new net PD2: U23.15 (D2)
- new net PD3: U23.17 (D3)
- new net PD4: U23.18 (D4)
- new net PD5: U23.19 (D5)
- new net PD6: U23.20 (D6)
- new net PD7: U23.21 (D7)
- new net RA0: U23.12 (A0)
- new net RA1: U23.11 (A1)
- new net RA2: U23.10 (A2)
- new net RA3: U23.9 (A3)
Other:
- note added: "FONT ROM"
- moved on the sheet: U19A, U19B, U20A, U20B, U21B, U22A, U22B

Commit message: Final work for rev 1
Parts:
- removed R26: 0R, COMET_footprints:R_SMD0805, symbol COMET_symbols:R
- removed unit 2 of U19
- removed U20: IS61C6416AL-12TLI, COMET_footprints:Package_TSOP-II-44_10.16x18.41mm_P0.8mm, symbol Video_Card:IS61C6416AL-12TLI
- removed U21: SN74LVC1G19DBV, COMET_footprints:Package_SOT23-6, symbol COMET_symbols:74x1G19
- removed unit 2 of U22
- removed U23: SST39SF010A-70-4C-NHE, COMET_footprints:Package_PLCC-32_SMD_socket, symbol COMET_symbols:39SF040
- renumbered U19 to U14, U22 to U15
Connections:
- net ~{B0CS}: now also U14.6 (~{CE})
Other:
- note removed: "FONT ROM"
